Commit message: starting the robot 3d model

File: src/simulation_pkg/urdf/caramelo.urdf (robot description, URDF)
Before this commit: robot caramelo, 1 links, 0 joints
Links:
- added link front_left_wheel; visual cylinder length=0.05 radius=0.05
- added link front_right_wheel; visual cylinder length=0.05 radius=0.05
- added link rear_left_wheel; visual cylinder length=0.05 radius=0.05
- added link rear_right_wheel; visual cylinder length=0.05 radius=0.05
- link base_link: geometry visual box size=0.530 0.220 0.150
Joints:
- added joint base_fl_wheel_joint: type fixed, parent base_link, child front_left_wheel, origin xyz=0.217 0.11 0 rpy=0 0 0
- added joint base_fr_wheel_joint: type fixed, parent base_link, child front_right_wheel, origin xyz=0.217 -0.11 0 rpy=0 0 0
- added joint base_rl_wheel_joint: type fixed, parent base_link, child rear_left_wheel, origin xyz=-0.217 0.11 0 rpy=0 0 0
- added joint base_rr_wheel_joint: type fixed, parent base_link, child rear_right_wheel, origin xyz=-0.217 -0.11 0 rpy=0 0 0

Commit message: add wheels to urdf file

File: src/simulation_pkg/urdf/caramelo.urdf (robot description, URDF)
Before this commit: robot caramelo, 5 links, 4 joints
Joints:
- joint base_fl_wheel_joint: axis (none) -> 0 0 1; origin xyz=0.217 0.11 0 rpy=0 0 0 -> xyz=0.217 0.11 0 rpy=-1.57 0 0; type fixed -> continuous
- joint base_fr_wheel_joint: axis (none) -> 0 0 1; origin xyz=0.217 -0.11 0 rpy=0 0 0 -> xyz=0.217 -0.11 0 rpy=1.57 0 0; type fixed -> continuous
- joint base_rl_wheel_joint: axis (none) -> 0 0 1; origin xyz=-0.217 0.11 0 rpy=0 0 0 -> xyz=-0.217 0.11 0 rpy=-1.57 0 0; type fixed -> continuous
- joint base_rr_wheel_joint: axis (none) -> 0 0 1; origin xyz=-0.217 -0.11 0 rpy=0 0 0 -> xyz=-0.217 -0.11 0 rpy=1.57 0 0; type fixed -> continuous
